Commit message: Completed urdf

File: config/so101_ros2_control.urdf.xacro (robot description, xacro)
@@ -2,32 +2,28 @@
 <!--
   so101_ros2_control.urdf.xacro
-  Include this inside your main robot URDF/xacro.
-  Each joint maps to one Waveshare ST servo via the 'servo_id' parameter.
+  Generated using onshape-to-robot
+  Onshape https://cad.onshape.com/documents/7715cc284bb430fe6dab4ffd/w/4fd0791b683777b02f8d975a/e/826c553ede3b7592eb9ca800
   Servo IDs must match the IDs programmed into the physical servos.
-  Default factory ID is 1. Use the Waveshare serial debug tool or
-  the SCServo SDK example 'ChangeID' to assign unique IDs per servo.
+  Default factory ID is 1. Use the Waveshare serial debug tool to assign unique IDs per servo.
 -->
 <robot xmlns:xacro="http://www.ros.org/wiki/xacro" name="so101">
+  <!-- ══════════════════════════════════════════════════════════════
+       ros2_control hardware interface
+       ══════════════════════════════════════════════════════════════ -->
   <ros2_control name="So101HardwareInterface" type="system">
     <hardware>
       <plugin>so101_hardware_interface/So101HardwareInterface</plugin>
-      <!-- ── Connection parameters ──────────────────────────────────── -->
-      <!-- USB serial port exposed by the Waveshare Bus Servo Adapter    -->
-      <param name="device_port">/dev/ttyUSB0</param>
-      <!-- ST-series default baud rate: 1 000 000                       -->
+      <!-- USB serial port exposed by the Waveshare Bus Servo Adapter -->
+      <param name="device_port">/dev/ttyACM0</param>
+      <!-- ST-series default baud rate: 1 000 000 -->
       <param name="baud_rate">1000000</param>
-      <!-- Comm timeout in seconds                                       -->
+      <!-- Comm timeout in seconds -->
       <param name="timeout">1.0</param>
-      <!-- ── Motion parameters ─────────────────────────────────────── -->
-      <!-- Speed in raw steps/s (0 = max servo speed, ~2400 typical)    -->
+      <!-- Speed in raw steps/s (0 = max servo speed, ~2400 typical) -->
       <param name="default_speed">0</param>
-      <!-- Acceleration 0–254 (0 = no limit)                            -->
+      <!-- Acceleration 0–254 (0 = no limit) -->
       <param name="default_acc">50</param>
     </hardware>
-    <!-- ── Joints ─────────────────────────────────────────────────────
-         servo_id: matches the ID burned into each physical servo (1-253)
-         min/max:  position limits in radians
-                   ST3215 full range = ±π  (raw 0–4095, centre = 2048)
-    ──────────────────────────────────────────────────────────────────── -->
+    <!-- Joint 1 → base→shoulder (shoulder pan) -->
     <joint name="shoulder_pan_joint">
       <param name="servo_id">1</param>
@@ -39,4 +35,5 @@
       <state_interface name="velocity"/>
     </joint>
+    <!-- Joint 2 → shoulder→upper_arm (shoulder lift) -->
     <joint name="shoulder_lift_joint">
       <param name="servo_id">2</param>
@@ -48,4 +45,5 @@
       <state_interface name="velocity"/>
     </joint>
+    <!-- Joint 3 → upper_arm→lower_arm (elbow flex) -->
     <joint name="elbow_flex_joint">
       <param name="servo_id">3</param>
@@ -57,4 +55,5 @@
       <state_interface name="velocity"/>
     </joint>
+    <!-- Joint 4 → lower_arm→wrist (wrist flex) -->
     <joint name="wrist_flex_joint">
       <param name="servo_id">4</param>
@@ -66,4 +65,5 @@
       <state_interface name="velocity"/>
     </joint>
+    <!-- Joint 5 → wrist→gripper (wrist roll) -->
     <joint name="wrist_roll_joint">
       <param name="servo_id">5</param>
@@ -75,4 +75,5 @@
       <state_interface name="velocity"/>
     </joint>
+    <!-- Joint 6 → gripper→moving_jaw (gripper) -->
     <joint name="gripper_joint">
       <param name="servo_id">6</param>
@@ -85,3 +86,415 @@
     </joint>
   </ros2_control>
+  <!-- ══════════════════════════════════════════════════════════════
+       Links
+       ══════════════════════════════════════════════════════════════ -->
+  <!-- Link base -->
+  <link name="base">
+    <inertial>
+      <origin xyz="-0.14932 -0.16812 0.065966" rpy="0 0 0"/>
+      <mass value="0.147"/>
+      <inertia ixx="0.000114686" ixy="-4.59787e-07" ixz="4.97151e-06" iyy="0.000136117" iyz="9.75275e-08" izz="0.000130364"/>
+    </inertial>
+    <!-- Part base_motor_holder_so101_v1 -->
+    <visual>
+      <origin xyz="-0.169402 -0.168167 0.0300817" rpy="1.5708 -1.67685e-15 1.5708"/>
+      <geometry>
+        <mesh filename="assets/base_motor_holder_so101_v1.stl"/>
+      </geometry>
+      <material name="base_motor_holder_so101_v1_material">
+        <color rgba="0.964706 0.964706 0.952941 1.0"/>
+      </material>
+    </visual>
+    <collision>
+      <origin xyz="-0.169402 -0.168167 0.0300817" rpy="1.5708 -1.67685e-15 1.5708"/>
+      <geometry>
+        <mesh filename="assets/base_motor_holder_so101_v1.stl"/>
+      </geometry>
+    </collision>
+    <!-- Part base_so101_v2 -->
+    <visual>
+      <origin xyz="-0.169402 -0.168068 0.0300817" rpy="1.5708 -1.6144e-15 1.5708"/>
+      <geometry>
+        <mesh filename="assets/base_so101_v2.stl"/>
+      </geometry>
+      <material name="base_so101_v2_material">
+        <color rgba="0.964706 0.964706 0.952941 1.0"/>
+      </material>
+    </visual>
+    <collision>
+      <origin xyz="-0.169402 -0.168068 0.0300817" rpy="1.5708 -1.6144e-15 1.5708"/>
+      <geometry>
+        <mesh filename="assets/base_so101_v2.stl"/>
+      </geometry>
+    </collision>
+    <!-- Part sts3215_03a_v1 -->
+    <visual>
+      <origin xyz="-0.136702 -0.168068 0.0761817" rpy="-8.21148e-16 7.84513e-18 1.249e-15"/>
+      <geometry>
+        <mesh filename="assets/sts3215_03a_v1.stl"/>
+      </geometry>
+      <material name="sts3215_03a_v1_material">
+        <color rgba="0.627451 0.627451 0.627451 1.0"/>
+      </material>
+    </visual>
+    <collision>
+      <origin xyz="-0.136702 -0.168068 0.0761817" rpy="-8.21148e-16 7.84513e-18 1.249e-15"/>
+      <geometry>
+        <mesh filename="assets/sts3215_03a_v1.stl"/>
+      </geometry>
+    </collision>
+    <!-- Part waveshare_mounting_plate_so101_v2 -->
+    <visual>
+      <origin xyz="-0.19402 -0.168267 0.0798817" rpy="1.5708 -1.35493e-14 1.5708"/>
+      <geometry>
+        <mesh filename="assets/waveshare_mounting_plate_so101_v2.stl"/>
+      </geometry>
+      <material name="waveshare_mounting_plate_so101_v2_material">
+        <color rgba="0.964706 0.964706 0.952941 1.0"/>
+      </material>
+    </visual>
+    <collision>
+      <origin xyz="-0.19402 -0.168267 0.0798817" rpy="1.5708 -1.35493e-14 1.5708"/>
+      <geometry>
+        <mesh filename="assets/waveshare_mounting_plate_so101_v2.stl"/>
+      </geometry>
+    </collision>
+  </link>
+  <!-- Frame baseframe (dummy link + fixed joint) -->
+  <link name="baseframe">
+    <origin xyz="0 0 0" rpy="0 -0 0"/>
+    <inertial>
+      <origin xyz="0 0 0" rpy="0 0 0"/>
+      <mass value="1e-9"/>
+      <inertia ixx="0" ixy="0" ixz="0" iyy="0" iyz="0" izz="0"/>
+    </inertial>
+  </link>
+  <joint name="baseframe_frame" type="fixed">
+    <origin xyz="-0.163038 -0.168068 0.0324817" rpy="1.6144e-15 7.84513e-18 1.33799e-15"/>
+    <parent link="base"/>
+    <child link="baseframe"/>
+    <axis xyz="0 0 0"/>
+  </joint>
+  <!-- Link shoulder -->
+  <link name="shoulder">
+    <inertial>
+      <origin xyz="-0.0307604 -1.66727e-05 -0.0252713" rpy="0 0 0"/>
+      <mass value="0.100006"/>
+      <inertia ixx="8.3759e-05" ixy="7.55525e-08" ixz="-1.16342e-06" iyy="8.10403e-05" iyz="1.54663e-07" izz="2.39783e-05"/>
+    </inertial>
+    <!-- Part sts3215_03a_v1_2 -->
+    <visual>
+      <origin xyz="-0.0303992 0.000422241 -0.0417" rpy="1.5708 1.5708 0"/>
+      <geometry>
+        <mesh filename="assets/sts3215_03a_v1.stl"/>
+      </geometry>
+      <material name="sts3215_03a_v1_2_material">
+        <color rgba="0.627451 0.627451 0.627451 1.0"/>
+      </material>
+    </visual>
+    <collision>
+      <origin xyz="-0.0303992 0.000422241 -0.0417" rpy="1.5708 1.5708 0"/>
+      <geometry>
+        <mesh filename="assets/sts3215_03a_v1.stl"/>
+      </geometry>
+    </collision>
+    <!-- Part motor_holder_so101_base_v1 -->
+    <visual>
+      <origin xyz="-0.0675992 -0.000177759 0.0158499" rpy="1.5708 -1.5708 0"/>
+      <geometry>
+        <mesh filename="assets/motor_holder_so101_base_v1.stl"/>
+      </geometry>
+      <material name="motor_holder_so101_base_v1_material">
+        <color rgba="0.964706 0.964706 0.952941 1.0"/>
+      </material>
+    </visual>
+    <collision>
+      <origin xyz="-0.0675992 -0.000177759 0.0158499" rpy="1.5708 -1.5708 0"/>
+      <geometry>
+        <mesh filename="assets/motor_holder_so101_base_v1.stl"/>
+      </geometry>
+    </collision>
+    <!-- Part rotation_pitch_so101_v1 -->
+    <visual>
+      <origin xyz="0.0122008 2.22413e-05 0.0464" rpy="-1.5708 2.35221e-33 0"/>
+      <geometry>
+        <mesh filename="assets/rotation_pitch_so101_v1.stl"/>
+      </geometry>
+      <material name="rotation_pitch_so101_v1_material">
+        <color rgba="0.964706 0.964706 0.952941 1.0"/>
+      </material>
+    </visual>
+    <collision>
+      <origin xyz="0.0122008 2.22413e-05 0.0464" rpy="-1.5708 2.35221e-33 0"/>
+      <geometry>
+        <mesh filename="assets/rotation_pitch_so101_v1.stl"/>
+      </geometry>
+    </collision>
+  </link>
+  <!-- Link upper_arm -->
+  <link name="upper_arm">
+    <inertial>
+      <origin xyz="-0.0898471 -0.00838224 0.0184089" rpy="0 0 0"/>
+      <mass value="0.103"/>
+      <inertia ixx="4.08002e-05" ixy="-1.97819e-05" ixz="-4.03016e-08" iyy="0.000147318" iyz="8.97326e-09" izz="0.000142487"/>
+    </inertial>
+    <!-- Part sts3215_03a_v1_3 -->
+    <visual>
+      <origin xyz="-0.11257 -0.0155 0.0187" rpy="-3.14159 -5.27356e-16 -1.5708"/>
+      <geometry>
+        <mesh filename="assets/sts3215_03a_v1.stl"/>
+      </geometry>
+      <material name="sts3215_03a_v1_3_material">
+        <color rgba="0.627451 0.627451 0.627451 1.0"/>
+      </material>
+    </visual>
+    <collision>
+      <origin xyz="-0.11257 -0.0155 0.0187" rpy="-3.14159 -5.27356e-16 -1.5708"/>
+      <geometry>
+        <mesh filename="assets/sts3215_03a_v1.stl"/>
+      </geometry>
+    </collision>
+    <!-- Part upper_arm_so101_v1 -->
+    <visual>
+      <origin xyz="-0.065085 0.012 0.0182" rpy="3.14159 -0 -1.30911e-30"/>
+      <geometry>
+        <mesh filename="assets/upper_arm_so101_v1.stl"/>
+      </geometry>
+      <material name="upper_arm_so101_v1_material">
+        <color rgba="0.964706 0.964706 0.952941 1.0"/>
+      </material>
+    </visual>
+    <collision>
+      <origin xyz="-0.065085 0.012 0.0182" rpy="3.14159 -0 -1.30911e-30"/>
+      <geometry>
+        <mesh filename="assets/upper_arm_so101_v1.stl"/>
+      </geometry>
+    </collision>
+  </link>
+  <!-- Link lower_arm -->
+  <link name="lower_arm">
+    <inertial>
+      <origin xyz="-0.0980701 0.00324376 0.0182831" rpy="0 0 0"/>
+      <mass value="0.104"/>
+      <inertia ixx="2.87438e-05" ixy="7.41152e-06" ixz="1.26409e-06" iyy="0.000159844" iyz="-4.90188e-08" izz="0.00014529"/>
+    </inertial>
+    <!-- Part under_arm_so101_v1 -->
+    <visual>
+      <origin xyz="-0.0648499 -0.032 0.0182" rpy="3.14159 -0 6.67202e-31"/>
+      <geometry>
+        <mesh filename="assets/under_arm_so101_v1.stl"/>
+      </geometry>
+      <material name="under_arm_so101_v1_material">
+        <color rgba="0.964706 0.964706 0.952941 1.0"/>
+      </material>
+    </visual>
+    <collision>
+      <origin xyz="-0.0648499 -0.032 0.0182" rpy="3.14159 -0 6.67202e-31"/>
+      <geometry>
+        <mesh filename="assets/under_arm_so101_v1.stl"/>
+      </geometry>
+    </collision>
+    <!-- Part motor_holder_so101_wrist_v1 -->
+    <visual>
+      <origin xyz="-0.0648499 -0.032 0.018" rpy="-3.14159 -2.55351e-15 -2.56146e-31"/>
+      <geometry>
+        <mesh filename="assets/motor_holder_so101_wrist_v1.stl"/>
+      </geometry>
+      <material name="motor_holder_so101_wrist_v1_material">
+        <color rgba="0.964706 0.964706 0.952941 1.0"/>
+      </material>
+    </visual>
+    <collision>
+      <origin xyz="-0.0648499 -0.032 0.018" rpy="-3.14159 -2.55351e-15 -2.56146e-31"/>
+      <geometry>
+        <mesh filename="assets/motor_holder_so101_wrist_v1.stl"/>
+      </geometry>
+    </collision>
+    <!-- Part sts3215_03a_v1_4 -->
+    <visual>
+      <origin xyz="-0.1224 0.0052 0.0187" rpy="-3.14159 -7.88861e-31 -3.14159"/>
+      <geometry>
+        <mesh filename="assets/sts3215_03a_v1.stl"/>
+      </geometry>
+      <material name="sts3215_03a_v1_4_material">
+        <color rgba="0.627451 0.627451 0.627451 1.0"/>
+      </material>
+    </visual>
+    <collision>
+      <origin xyz="-0.1224 0.0052 0.0187" rpy="-3.14159 -7.88861e-31 -3.14159"/>
+      <geometry>
+        <mesh filename="assets/sts3215_03a_v1.stl"/>
+      </geometry>
+    </collision>
+  </link>
+  <!-- Link wrist -->
+  <link name="wrist">
+    <inertial>
+      <origin xyz="-0.000103312 -0.0386143 0.0281156" rpy="0 0 0"/>
+      <mass value="0.079"/>
+      <inertia ixx="3.68263e-05" ixy="1.7893e-08" ixz="-5.28128e-08" iyy="2.5391e-05" iyz="3.6412e-06" izz="2.1e-05"/>
+    </inertial>
+    <!-- Part sts3215_03a_no_horn_v1 -->
+    <visual>
+      <origin xyz="5.55112e-17 -0.0424 0.0306" rpy="1.5708 1.5708 0"/>
+      <geometry>
+        <mesh filename="assets/sts3215_03a_no_horn_v1.stl"/>
+      </geometry>
+      <material name="sts3215_03a_no_horn_v1_material">
+        <color rgba="0.627451 0.627451 0.627451 1.0"/>
+      </material>
+    </visual>
+    <collision>
+      <origin xyz="5.55112e-17 -0.0424 0.0306" rpy="1.5708 1.5708 0"/>
+      <geometry>
+        <mesh filename="assets/sts3215_03a_no_horn_v1.stl"/>
+      </geometry>
+    </collision>
+    <!-- Part wrist_roll_pitch_so101_v2 -->
+    <visual>
+      <origin xyz="0 -0.028 0.0181" rpy="-1.5708 -1.5708 0"/>
+      <geometry>
+        <mesh filename="assets/wrist_roll_pitch_so101_v2.stl"/>
+      </geometry>
+      <material name="wrist_roll_pitch_so101_v2_material">
+        <color rgba="0.964706 0.964706 0.952941 1.0"/>
+      </material>
+    </visual>
+    <collision>
+      <origin xyz="0 -0.028 0.0181" rpy="-1.5708 -1.5708 0"/>
+      <geometry>
+        <mesh filename="assets/wrist_roll_pitch_so101_v2.stl"/>
+      </geometry>
+    </collision>
+  </link>
+  <!-- Link gripper -->
+  <link name="gripper">
+    <inertial>
+      <origin xyz="0.000213627 0.000245138 -0.025187" rpy="0 0 0"/>
+      <mass value="0.087"/>
+      <inertia ixx="2.75087e-05" ixy="-3.35241e-07" ixz="-5.7352e-06" iyy="4.33657e-05" iyz="-5.17847e-08" izz="3.45059e-05"/>
+    </inertial>
+    <!-- Part sts3215_03a_v1_5 -->
+    <visual>
+      <origin xyz="0.0077 0.0001 -0.0234" rpy="-1.5708 -5.19179e-17 -1.66533e-16"/>
+      <geometry>
+        <mesh filename="assets/sts3215_03a_v1.stl"/>
+      </geometry>
+      <material name="sts3215_03a_v1_5_material">
+        <color rgba="0.627451 0.627451 0.627451 1.0"/>
+      </material>
+    </visual>
+    <collision>
+      <origin xyz="0.0077 0.0001 -0.0234" rpy="-1.5708 -5.19179e-17 -1.66533e-16"/>
+      <geometry>
+        <mesh filename="assets/sts3215_03a_v1.stl"/>
+      </geometry>
+    </collision>
+    <!-- Part wrist_roll_follower_so101_v1 -->
+    <visual>
+      <origin xyz="0 -0.000218214 0.000949706" rpy="-3.14159 -5.55112e-17 0"/>
+      <geometry>
+        <mesh filename="assets/wrist_roll_follower_so101_v1.stl"/>
+      </geometry>
+      <material name="wrist_roll_follower_so101_v1_material">
+        <color rgba="0.964706 0.964706 0.952941 1.0"/>
+      </material>
+    </visual>
+    <collision>
+      <origin xyz="0 -0.000218214 0.000949706" rpy="-3.14159 -5.55112e-17 0"/>
+      <geometry>
+        <mesh filename="assets/wrist_roll_follower_so101_v1.stl"/>
+      </geometry>
+    </collision>
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